File: schematics/arithmetic-logic-unit/arithmetic-logic-unit.kicad_sch (KiCad schematic)
At the start: 102 parts, among them U1 74LS151, U10 AT28C64B-15PC, U11 74LS32, U12 74LS32, U13 74LS32, U14 74LS32, U15 74LS32, U16 74LS32, U17 74LS32, U18 74LS32, U19 74LS86, U2 74LS151, U20 74LS86, U21 74LS86, U22 74LS86, U23 74LS86, U24 74LS86, U25 74LS86, U26 74LS86, U27 74LS574, U28 74LS86, U29 74LS245, U3 74LS151, U31 74LS08, U32 74LS08, U33 74LS08, U34 74LS08, U35 74LS08, U36 74LS08, U37 74LS32, U38 74LS86, U39 74LS86, U4 74LS151, U40 74LS86, U41 74LS86, U42 74LS86, U43 74LS86, U44 74LS86, U45 74LS86, U46 74LS86, U47 74LS08, U48 74LS08, U49 74LS08, U5 74LS151, U50 74LS08, U51 74LS08, U52 74LS08, U53 74LS08, U54 74LS08, U55 74LS08, U56 74LS08, U57 74LS08, U58 74LS08, U59 74LS08, U6 74LS151, U60 74LS08, U61 74LS08, U62 74LS08, U63 74LS08, U64 74LS32, U65 74LS32, U66 74LS32, U67 74LS32, U68 74LS32, U69 74LS32, U7 74LS151, U70 74LS32, U71 74LS32, U8 74LS151, U9 74LS245

Commit message: Corrected ALU schematic after diy pcb soldered
Parts:
- removed unit 4 of U31
- removed unit 4 of U32
- removed unit 4 of U33
- removed unit 4 of U34
- removed unit 4 of U35
- removed unit 4 of U36
- removed U63: 74LS08, symbol 74xx:74LS08
- added U30, U63, U72, U73, U74, U75, U76: 74LS32, symbol 74xx:74LS32
- added unit 1 of U46
- added U77, U78, U79, U80, U81, U82, U83: 74LS86, symbol 74xx:74LS86
Connections:
- net +5V: now also U1.3 (I1), U2.3 (I1), U3.3 (I1), U4.3 (I1), U5.3 (I1), U6.3 (I1), U7.3 (I1), U8.3 (I1), U8.4 (I0)
- net GND: now also U1.12 (I7), U1.4 (I0), U2.4 (I0), U3.4 (I0), U4.4 (I0), U5.4 (I0), U6.4 (I0), U7.4 (I0), U8.14 (I5); no longer U10.6 (A4)
- net at U12.1, U32.4, U39.1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: now also U77.1; no longer U2.3 (I1)
- net at U12.2, U32.5, U39.2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: now also U77.2; no longer U2.2 (I2)
- net at R17.1, U1.5 (Z), U27.2 (D0)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: now also U30.1
- net at U17.1, U44.1, U47.4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: now also U82.1; no longer U7.3 (I1)
- net at U17.2, U44.2, U47.5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: now also U82.2; no longer U7.2 (I2)
- net at U18.2, U45.2, U48.5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: now also U83.2; no longer U8.2 (I2)
- net at U7.12 (I7): now also U24.6, U5.14 (I5), U6.2 (I2), U7.13 (I6)
- net at U7.14 (I5): now also U26.6, U8.2 (I2)
- net at U7.15 (I4): now also U82.3
- net at U25.6: now also U6.14 (I5), U7.2 (I2), U8.12 (I7), U8.13 (I6); no longer U7.4 (I0)
- net at R23.1, U7.5 (Z), U9.3 (A1): now also U73.1
- net at R20.1, U4.5 (Z), U9.6 (A4): now also U63.2
- net at R19.1, U3.5 (Z), U9.7 (A5): now also U63.1
- net at U2.12 (I7): now also U1.13 (I6), U1.2 (I2), U19.6, U2.13 (I6)
- net at U2.14 (I5): now also U21.6, U3.2 (I2), U4.12 (I7), U4.13 (I6)
- net at U2.15 (I4): now also U77.3
- net at U20.6: now also U1.14 (I5), U2.2 (I2), U3.12 (I7), U3.13 (I6); no longer U2.4 (I0)
- net at R18.1, U2.5 (Z), U9.8 (A6): now also U30.2
- net at U16.1, U36.4, U43.1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: now also U81.1; no longer U6.3 (I1)
- net at U16.2, U36.5, U43.2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: now also U81.2; no longer U6.2 (I2)
- net at U15.1, U35.4, U42.1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: now also U80.1; no longer U5.3 (I1)
- net at U15.2, U35.5, U42.2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: now also U80.2; no longer U5.2 (I2)
- net at U18.1, U45.1, U48.4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: now also U83.1; no longer U8.3 (I1)
- net at U14.1, U34.4, U41.1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: now also U79.1; no longer U4.3 (I1)
- net at U13.2, U33.5, U40.2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: now also U78.2; no longer U3.2 (I2)
- net at R22.1, U6.5 (Z), U9.4 (A2): now also U72.2
- net at U3.14 (I5): now also U22.6, U4.2 (I2), U5.12 (I7), U5.13 (I6)
- net at U3.15 (I4): now also U78.3
- net at U13.1, U33.4, U40.1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: now also U78.1; no longer U3.3 (I1)
- net at R21.1, U5.5 (Z), U9.5 (A3): now also U72.1
- net at R24.1, U27.3 (D1), U8.5 (Z)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: now also U73.2
- net at U8.15 (I4): now also U83.3
- net at U4.14 (I5): now also U23.6, U5.2 (I2), U6.12 (I7), U6.13 (I6)
- net at U4.15 (I4): now also U79.3
- net at U14.2, U34.5, U41.2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: now also U79.2; no longer U4.2 (I2)
- net at U5.15 (I4): now also U80.3
- net at U27.4 (D2): now also U76.3
- net at U11.2, U31.5, U38.2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: now also U46.2; no longer U1.2 (I2)
- net at U1.15 (I4): now also U46.3
- net at U11.1, U31.4, U38.1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: now also U46.1; no longer U1.3 (I1)
- net at U6.15 (I4): now also U81.3
- net INV_(A_OR_B) renamed INV_OR_RESULT
- net ~{FLAGS_OUT} renamed ~{REG_F_OUT}
- new net: U30.3, U74.1
- new net: U72.3, U75.1
- new net: U74.3, U76.1
- new net: U75.3, U76.2
- new net: U63.3, U74.2
- new net: U73.3, U75.2
- new net ALU_OPC_4: U10.6 (A4)
Other:
- moved on the sheet: U11A, U12A, U13A, U14A, U15A, U16A, U17A, U18A, U19A, U19B, U20A, U20B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

Commit message: Schematics and interrupts
Connections:
- net GND: no longer U27.11 (Cp)
- new net REG_F_LOAD: U27.11 (Cp)
