File: schematics/control-unit/control-unit.kicad_sch (KiCad schematic)
At the start: 58 parts, among them SW1 SW_DPDT_x2, SW2 SW_Push, SW3 SW_Push, SW4 SW_Push, U1 AT28C64B-15PC, U10 74LS08, U11 74LS08, U13 74LS161, U14 74LS574, U15 74LS08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

Commit message: Control unit build
Parts:
- removed R8 (x3): R_US, symbol Device:R_US
- removed SW2, SW3, SW4: SW_Push, symbol Switch:SW_Push
- removed U11: 74LS08, symbol 74xx:74LS08
- added U12: 74LS08, symbol 74xx:74LS08
Connections:
- net ADDRESS_DIR is gone; now on net ~{ALU_OUT}: U23.18 (Q1)
- net MAR_LOAD is gone; now on net PC_TICK: U20.3
- net WORD_DIR is gone; now on net ~{STC_LOAD}: U36.19 (Q0)
- net ~{MAN_INPUT} is gone; now on net ~{STC_OUT}: U36.15 (Q4)
- net ~{MAR_OUT} is gone; now on net ~{PC_LOAD}: U32.15 (Q4)
- net ~{MBR_OUT} is gone; now on net ~{PC_RST}: U32.14 (Q5)
- net ~{PASS_DATA} is gone; now on net ALU_OPC_4: U7.13 (Q6)
- net ~{PASS_WORD} is gone; now on net STC_RST: U36.18 (Q1)
- net ~{TMP_H_OUT} is gone; now on net ALU_OPC_2: U7.15 (Q4)
- net ~{TMP_L_OUT} is gone; now on net ALU_OPC_3: U7.14 (Q5)
- net +5V: now also U13.1 (~{MR})
- net ALU_OPC_0: now also U7.17 (Q2); no longer U23.17 (Q2)
- net ALU_OPC_1: now also U7.16 (Q3); no longer U23.16 (Q3)
- net ALU_OPC_2: no longer U23.15 (Q4)
- net ALU_OPC_3: no longer U23.14 (Q5)
- net ALU_OPC_4: no longer U23.13 (Q6)
- net CLK: now also U12.1; no longer U20.1, U23.11 (Cp), U32.11 (Cp), U36.11 (Cp), U37.11 (Cp), U38.11 (Cp), U7.11 (Cp)
- net MCC_TICK: now also U10.3
- net MEM_PART: now also U37.18 (Q1); no longer U36.17 (Q2)
- net PC_TICK: no longer U8.3
- net STC_MODE: now also U36.16 (Q3); no longer U37.17 (Q2)
- net STC_TICK: now also U8.3; no longer U9.3
- net ~{ALU_OUT}: no longer U32.18 (Q1)
- net ~{CLK}: now also U20.1, U23.11 (Cp), U32.11 (Cp), U36.11 (Cp), U37.11 (Cp), U38.11 (Cp), U7.11 (Cp)
- net ~{MCC_RST}: now also U38.17 (Q2); no longer U37.13 (Q6)
- net ~{MEM_IN}: now also U37.19 (Q0); no longer U32.12 (Q7)
- net ~{MEM_OUT}: now also U36.12 (Q7); no longer U32.13 (Q6)
- net ~{PC_LOAD}: no longer U36.14 (Q5)
- net ~{PC_OUT}: now also U32.12 (Q7); no longer U36.12 (Q7)
- net ~{STC_LOAD}: no longer U37.19 (Q0)
- net ~{STC_OUT}: no longer U37.16 (Q3)
- net ~{ZERO_PAGE}: now also U37.17 (Q2); no longer U36.16 (Q3)
- net at U19.2: now also U36.14 (Q5); no longer U23.12 (Q7)
- net at U8.2: now also U36.17 (Q2); no longer U36.13 (Q6)
- net ~{REG_MBR_USE_BTTNS}: now reaches U37.14 (Q5)
- net at U10.2: now also U38.18 (Q1); no longer U37.15 (Q4)
- net at U9.2: now also U38.19 (Q0); no longer U37.18 (Q1)
- net at U21.2: now also U36.13 (Q6); no longer U32.16 (Q3)
- net at U20.2: now also U32.13 (Q6); no longer U32.17 (Q2)
- net at U18.2: now also U23.16 (Q3); no longer U7.16 (Q3)
- net at U17.2: now also U23.17 (Q2); no longer U7.17 (Q2)
- net DATA_DIR renamed ~{REG_F_OUT}
- net FLAGS_LOAD renamed REG_MAR_LOAD
- net IR_LOAD renamed REG_IR_LOAD
- net REG_IR_LOAD: now also U9.3; no longer U10.3
- net MBR_LOAD renamed REG_MBR_LOAD
- net TMP_H_LOAD renamed REG_TMPH_LOAD
- net TMP_L_LOAD renamed REG_TMPL_LOAD
- net ~{FLAGS_OUT} renamed ~{REG_TMPL_PASS_DATA}
- net ~{PASS_ADDRESS}: no longer names the net of U7.12 (Q7)
- net ~{PASS_ADDRESS}: now also U12.2
- new net REG_F_LOAD: U12.3
- new net REG_MBR_WORD_DIR: U37.16 (Q3)
- new net REG_TMPH_DATA_DIR: U32.17 (Q2)
- new net REG_TMPL_DATA_DIR: U32.16 (Q3)
- new net REG_TMP_ADDRESS_DIR: U32.18 (Q1)
- new net ~{REG_MAR_USE_BTTNS}: U37.15 (Q4)
- new net ~{REG_MBR_USE_BUS}: U37.13 (Q6)
- new net ~{REG_TMPH_OUT}: U23.15 (Q4)
- new net ~{REG_TMPH_PASS_DATA}: U23.12 (Q7)
- new net ~{REG_TMPL_OUT}: U23.14 (Q5)
- new net ~{REG_TMP_PASS_ADDRESS}: U23.13 (Q6)
- no-connect marks 11 -> 8
Other:
- moved on the sheet: U15A, U16A, U17A, U18A, U20A, U23, U7, U8A
