File: schematics/memory-unit/memory-unit.kicad_sch (KiCad schematic)
At the start: 118 parts, among them SW1 SW_DIP_x08, SW2 SW_DIP_x08, SW3 SW_DIP_x08, U1 AS6C1008-55PCN, U10 74LS574, U11 74LS04, U12 74LS08, U13 74LS08, U14 74LS08, U15 74LS08, U16 74LS08, U17 74LS08, U18 74LS08, U19 74LS08, U2 74LS245, U3 74LS245, U4 74LS245, U5 74LS245, U6 74LS245, U7 74LS245, U8 74LS574, U9 74LS574

Commit message: Corrections after second diy pcb soldered
Parts:
- removed R8 (x24): R_US, symbol Device:R_US
- added U21, U22: 74LS245, symbol 74xx:74LS245
Connections:
- net ~{MAR_OUT} is gone; now on net GND: U10.1 (OE), U9.1 (OE)
- net ~{MBR_OUT} is gone; now on net GND: U8.1 (OE)
- net +5V: now also SW1.1, SW1.2, SW1.3, SW1.4, SW1.5, SW1.6, SW1.7, SW1.8, SW2.1, SW2.2, SW2.3, SW2.4, SW2.5, SW2.6, SW2.7, SW2.8, SW3.1, SW3.2, SW3.3, SW3.4, SW3.5, SW3.6, SW3.7, SW3.8, U21.1 (A->B), U21.20 (VCC), U22.20 (VCC); no longer R8.1, R8.1, R8.1, R8.1, R8.1, R8.1, R8.1, R8.1, R8.1, R8.1, R8.1, R8.1, R8.1, R8.1, R8.1, R8.1, R8.1, R8.1, R8.1, R8.1, R8.1, R8.1, R8.1, R8.1
- net GND: now also R8.1, R8.1, R8.1, R8.1, R8.1, R8.1, R8.1, R8.1, R8.1, R8.1, R8.1, R8.1, R8.1, R8.1, R8.1, R8.1, R8.1, R8.1, R8.1, R8.1, R8.1, R8.1, R8.1, R8.1, U21.10 (GND), U22.1 (A->B), U22.10 (GND)
- net ~{MEM_IN}: now also U21.19 (CE)
- net ~{MEM_OUT}: now also U22.19 (CE)
- net at U2.11 (B7), U3.11 (B7), U8.9 (D7): now also U22.9 (A7); no longer R1.1, U1.21 (DQ7), U8.12 (Q7)
- net at U2.18 (B0), U3.18 (B0), U8.2 (D0): now also U22.2 (A0); no longer R8.1, U1.13 (DQ0), U8.19 (Q0)
- net at U2.13 (B5), U3.13 (B5), U8.7 (D5): now also U22.7 (A5); no longer R3.1, U1.19 (DQ5), U8.14 (Q5)
- net at U2.12 (B6), U3.12 (B6), U8.8 (D6): now also U22.8 (A6); no longer R2.1, U1.20 (DQ6), U8.13 (Q6)
- net at U2.14 (B4), U3.14 (B4), U8.6 (D4): now also U22.6 (A4); no longer R4.1, U1.18 (DQ4), U8.15 (Q4)
- net at U2.15 (B3), U3.15 (B3), U8.5 (D3): now also U22.5 (A3); no longer R5.1, U1.17 (DQ3), U8.16 (Q3)
- net at U2.16 (B2), U3.16 (B2), U8.4 (D2): now also U22.4 (A2); no longer R6.1, U1.15 (DQ2), U8.17 (Q2)
- net at U2.17 (B1), U3.17 (B1), U8.3 (D1): now also U22.3 (A1); no longer R7.1, U1.14 (DQ1), U8.18 (Q1)
- net MAR_LOAD renamed REG_MAR_LOAD
- net MBR_LOAD renamed REG_MBR_LOAD
- net WORD_DIR renamed REG_MBR_WORD_DIR
- net ~{MAN_INPUT} renamed ~{REG_MAR_USE_BTTNS}
- net ~{REG_MAR_USE_BTTNS}: no longer U2.19 (CE)
- net ~{PASS_WORD} renamed ~{REG_MBR_USE_BUS}
- new net: R1.1, U1.21 (DQ7), U21.11 (B7), U22.11 (B7)
- new net: R8.1, U1.13 (DQ0), U21.18 (B0), U22.18 (B0)
- new net: R3.1, U1.19 (DQ5), U21.13 (B5), U22.13 (B5)
- new net: U21.9 (A7), U8.12 (Q7)
- new net: U21.8 (A6), U8.13 (Q6)
- new net: U21.7 (A5), U8.14 (Q5)
- new net: U21.6 (A4), U8.15 (Q4)
- new net: U21.5 (A3), U8.16 (Q3)
- new net: U21.4 (A2), U8.17 (Q2)
- new net: U21.3 (A1), U8.18 (Q1)
- new net: U21.2 (A0), U8.19 (Q0)
- new net: R4.1, U1.18 (DQ4), U21.14 (B4), U22.14 (B4)
- new net: R7.1, U1.14 (DQ1), U21.17 (B1), U22.17 (B1)
- new net: R6.1, U1.15 (DQ2), U21.16 (B2), U22.16 (B2)
- new net: R2.1, U1.20 (DQ6), U21.12 (B6), U22.12 (B6)
- new net: R5.1, U1.17 (DQ3), U21.15 (B3), U22.15 (B3)
- new net ~{REG_MBR_USE_BTTNS}: U2.19 (CE)
Other:
- moved on the sheet: R8, SW1, U1, U2, U3, U8
