File: schematics/program-counter/program-counter.kicad_sch (KiCad schematic)
At the start: 38 parts, among them U1 74LS161, U2 74LS161, U3 74LS161, U4 74LS245, U5 74LS161, U6 74LS245

Commit message: Corrections after second diy pcb soldered
Connections:
- net +5V: now also U5.10 (CET)
- net GND: no longer U1.15 (TC), U5.10 (CET)
- no-connect marks 0 -> 1
Changed lines of the file:
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@@
   (junction (at 227.33 99.06) (diameter 0) (color 0 0 0 0)
   )
-  (junction (at 237.49 146.05) (diameter 0) (color 0 0 0 0)
-  )
   (junction (at 120.65 157.48) (diameter 0) (color 0 0 0 0)
   )
@@
   (junction (at 82.55 16.51) (diameter 0) (color 0 0 0 0)
   )
+  (junction (at 208.28 125.73) (diameter 0) (color 0 0 0 0)
+  )
   (junction (at 100.33 16.51) (diameter 0) (color 0 0 0 0)
   )
@@
   (junction (at 223.52 53.34) (diameter 0) (color 0 0 0 0)
   )
-  (wire (pts (xy 86.36 109.22) (xy 86.36 125.73))
-    (stroke (width 0) (type default))
-  )
+  (no_connect (at 64.77 113.03))
   (wire (pts (xy 100.33 16.51) (xy 109.22 16.51))
     (stroke (width 0) (type default))
@@
     (stroke (width 0) (type default))
   )
+  (wire (pts (xy 237.49 139.7) (xy 237.49 138.43))
+    (stroke (width 0) (type default))
+  )
   (wire (pts (xy 176.53 157.48) (xy 120.65 157.48))
     (stroke (width 0) (type default))
@@
     (stroke (width 0) (type default))
   )
-  (wire (pts (xy 237.49 138.43) (xy 237.49 146.05))
-    (stroke (width 0) (type default))
-  )
   (wire (pts (xy 219.71 106.68) (xy 252.73 106.68))
     (stroke (width 0) (type default))
@@
     (stroke (width 0) (type default))
   )
+  (wire (pts (xy 208.28 139.7) (xy 208.28 125.73))
+    (stroke (width 0) (type default))
+  )
   (wire (pts (xy 223.52 49.53) (xy 223.52 53.34))
     (stroke (width 0) (type default))
@@
     (stroke (width 0) (type default))
   )
+  (wire (pts (xy 208.28 139.7) (xy 237.49 139.7))
+    (stroke (width 0) (type default))
+  )
   (wire (pts (xy 64.77 31.75) (xy 64.77 27.94))
     (stroke (width 0) (type default))
@@
     (stroke (width 0) (type default))
   )
-  (wire (pts (xy 234.95 146.05) (xy 237.49 146.05))
+  (wire (pts (xy 234.95 146.05) (xy 254 146.05))
     (stroke (width 0) (type default))
   )
@@
     (stroke (width 0) (type default))
   )
-  (wire (pts (xy 64.77 109.22) (xy 86.36 109.22))
-    (stroke (width 0) (type default))
-  )
   (wire (pts (xy 179.07 146.05) (xy 198.12 146.05))
     (stroke (width 0) (type default))
@@
     (stroke (width 0) (type default))
   )
-  (wire (pts (xy 237.49 146.05) (xy 254 146.05))
-    (stroke (width 0) (type default))
-  )
   (wire (pts (xy 96.52 121.92) (xy 96.52 125.73))
     (stroke (width 0) (type default))
@@
     (stroke (width 0) (type default))
   )
-  (wire (pts (xy 64.77 113.03) (xy 64.77 109.22))
-    (stroke (width 0) (type default))
-  )
