File: schematics/final-cu/final-cu.kicad_pcb (KiCad board)
At the start: 2 copper layers, 200 x 300 mm, 148 parts

Commit message: Improved details
Parts:
- added AND-GATE-INT2: CD4081BEE4, Package_DIP:DIP-14_W7.62mm, F.Cu at (-31.2, 240.5)
- added AND-GATE-INT3: CD4081BEE4, Package_DIP:DIP-14_W7.62mm, F.Cu at (-20.4, 240.5)
- moved EEPROM-SIGNALS-G1 395.4 mm to (-45.5, 180.2), turned to 0 degrees
- moved SR-LATCH_INTERRUPTS1 371.9 mm to (99.7, 232.2)
- moved SR-LATCH-INTERRUPTS2 365.3 mm to (99.7, 216.6)
- moved NOT-GATE-SELECTOR1 331.2 mm to (92.4, 172.1)
- moved BUFFER-G1 320.2 mm to (-49.9, 170.2)
- moved ENABLE-INTERRUPTS2 315.7 mm to (123.9, 216.6), turned to 90 degrees
- moved ENABLE-INTERRUPTS1 310.0 mm to (123.9, 232.2), turned to 90 degrees
- moved INTERRUPTS-IN1 264.9 mm to (81.2, 216.5)
- moved INTERRUPTS-IN2 264.9 mm to (81.1, 224.5)
- moved R_UP1 245.7 mm to (42.3, 173.8), turned to 0 degrees
- moved BOOT-MODE1 226.4 mm to (43.4, 163.3)
- moved INTERRUPTS-OUT1 217.2 mm to (299.2, 16.8)
- moved INTERRUPTS-OUT2 217.2 mm to (299.2, 25.0)
- moved LED_INT0 172.6 mm to (137.2, 190.6)
- moved LED_INT1 172.6 mm to (130.5, 190.6)
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- renumbered AND-GATE-INT-ADDRESS1 to AND-GATE-INT1, NOT-GATE-INT-ADDRESS1 to NOT-GATE-INT1, OR-GATE-INT-ADDRESS1 to OR-GATE-INT1
Connections:
- net INT_ADDRESS_OUT renamed ~{INT_ADDRESS_OUT}
- AND-GATE-INT1 pad 10: unconnected-(AND-GATE-INT-ADDRESS1-L=E.F-Pad10) -> INT_2``_AND_(~{INT_3``_OR_INT_4``})
- AND-GATE-INT1 pad 11: unconnected-(AND-GATE-INT-ADDRESS1-M=G.H-Pad11) -> INT_3``_AND_~{INT_4``}
- AND-GATE-INT1 pad 12: unconnected-(AND-GATE-INT-ADDRESS1-G-Pad12) -> ~{INT_4``}
- AND-GATE-INT1 pad 13: unconnected-(AND-GATE-INT-ADDRESS1-H-Pad13) -> INT_3``
- AND-GATE-INT1 pad 8: unconnected-(AND-GATE-INT-ADDRESS1-E-Pad8) -> ~{INT_3``_OR_INT_4``}
- AND-GATE-INT1 pad 9: unconnected-(AND-GATE-INT-ADDRESS1-F-Pad9) -> INT_2``
- BUFFER-G1 pad 12: RST_INT_4 -> unconnected-(BUFFER-G1-8Q-Pad12)
- BUFFER-G1 pad 13: RST_INT_3 -> unconnected-(BUFFER-G1-7Q-Pad13)
- BUFFER-G1 pad 14: RST_INT_2 -> unconnected-(BUFFER-G1-6Q-Pad14)
- BUFFER-G1 pad 15: RST_INT_1 -> unconnected-(BUFFER-G1-5Q-Pad15)
- BUFFER-G1 pad 16: RST_INT_0 -> unconnected-(BUFFER-G1-4Q-Pad16)
- NOT-GATE-INT1 pad 1: INT_3``_OR_INT_4`` -> INT_1``
- NOT-GATE-INT1 pad 10: unconnected-(NOT-GATE-INT-ADDRESS1-~{5Y}-Pad10) -> ~{INT_1``_OR_INT_2``}
- NOT-GATE-INT1 pad 11: unconnected-(NOT-GATE-INT-ADDRESS1-5A-Pad11) -> INT_1``_OR_INT_2``
- NOT-GATE-INT1 pad 12: unconnected-(NOT-GATE-INT-ADDRESS1-~{6Y}-Pad12) -> ~{INT_3``_OR_INT_4``}
- NOT-GATE-INT1 pad 13: unconnected-(NOT-GATE-INT-ADDRESS1-6A-Pad13) -> INT_3``_OR_INT_4``
- NOT-GATE-INT1 pad 2: ~{INT_3``_OR_INT_4``} -> ~{INT_1``}
- NOT-GATE-INT1 pad 3: INT_1`` -> INT_2``
- NOT-GATE-INT1 pad 4: ~{INT_1``} -> ~{INT_2``}
- NOT-GATE-INT1 pad 8: unconnected-(NOT-GATE-INT-ADDRESS1-~{4Y}-Pad8) -> ~{INT_4``}
- NOT-GATE-INT1 pad 9: unconnected-(NOT-GATE-INT-ADDRESS1-4A-Pad9) -> INT_4``
- OR-GATE-RESETS1 pad 10: unconnected-(OR-GATE-RESETS1-L=E+F-Pad10) -> RST_INT_ENABLE`
- OR-GATE-RESETS1 pad 8: unconnected-(OR-GATE-RESETS1-E-Pad8) -> RST_INT_ENABLE
- OR-GATE-RESETS1 pad 9: unconnected-(OR-GATE-RESETS1-F-Pad9) -> MASTER_RESET
- SR-LATCH-INTERRUPTS2 pad 3: RST_INT_ENABLE -> RST_INT_ENABLE`
- TRNS-INT-ADDRESS1 pad 11: ADDRESSS0 -> ADDRESS0
Routing:
- net IR7: track 0.00 -> 416.9 mm
- net IR4: track 0.00 -> 413.7 mm
- net IR5: track 0.00 -> 409.7 mm
- net IR6: track 0.00 -> 368.4 mm
- net MC1: track 0.00 -> 364.5 mm
- net MC0: track 0.00 -> 362.4 mm
- net MC2: track 0.00 -> 332.4 mm
- net MC3: track 0.00 -> 328.5 mm
- net IR0: track 0.00 -> 312.1 mm
- net IR1: track 0.00 -> 276.0 mm
- net IR2: track 0.00 -> 275.3 mm
- net IR3: track 0.00 -> 265.9 mm
- net MODE: track 0.00 -> 229.1 mm
- net INT_ENABLE: track 0.00 -> 107.6 mm
- net Net-(EEPROM-INTERRUPT-CHECK1-A0): track 0.00 -> 98.5 mm
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