File: schematics/final-cu/final-cu.kicad_sch (KiCad schematic)
At the start: 148 parts

Commit message: Improved details
Parts:
- added AND-GATE-INT2, AND-GATE-INT3: CD4081BEE4, Package_DIP:DIP-14_W7.62mm, symbol CD4081BEE4:CD4081BEE4
- renumbered AND-GATE-INT-ADDRESS1 to AND-GATE-INT1, NOT-GATE-INT-ADDRESS1 to NOT-GATE-INT1, OR-GATE-INT-ADDRESS1 to OR-GATE-INT1
Connections:
- net ADDRESSS0 is gone; now on net ADDRESS0: TRNS-INT-ADDRESS1.11 (B8)
- net GND: now also AND-GATE-INT2.7 (VSS), AND-GATE-INT3.7 (VSS)
- net INT_1``: now also NOT-GATE-INT1.1 (1A), AND-GATE-INT3.13 (H); no longer NOT-GATE-INT1.3 (2A)
- net INT_1``_OR_INT_2``: now also NOT-GATE-INT1.11 (5A)
- net INT_2``: now also AND-GATE-INT1.9 (F), NOT-GATE-INT1.3 (2A)
- net INT_3``: now also AND-GATE-INT1.13 (H)
- net INT_3``_OR_INT_4``: now also NOT-GATE-INT1.13 (6A); no longer NOT-GATE-INT1.1 (1A)
- net INT_4``: now also NOT-GATE-INT1.9 (4A), AND-GATE-INT2.1 (A)
- net MASTER_RESET: now also OR-GATE-RESETS1.9 (F)
- net RST_INT_0: now also AND-GATE-INT3.3 (J=A.B); no longer BUFFER-G1.16 (4Q)
- net RST_INT_1: now also AND-GATE-INT2.11 (M=G.H); no longer BUFFER-G1.15 (5Q)
- net RST_INT_2: now also AND-GATE-INT2.10 (L=E.F); no longer BUFFER-G1.14 (6Q)
- net RST_INT_3: now also AND-GATE-INT2.4 (K=C.D); no longer BUFFER-G1.13 (7Q)
- net RST_INT_4: now also AND-GATE-INT2.3 (J=A.B); no longer BUFFER-G1.12 (8Q)
- net RST_INT_ENABLE: now also OR-GATE-RESETS1.8 (E); no longer SR-LATCH-INTERRUPTS2.3 (R1)
- net SET_INT_ENABLE: now also AND-GATE-INT2.12 (G), AND-GATE-INT2.2 (B), AND-GATE-INT2.5 (C), AND-GATE-INT2.9 (F), AND-GATE-INT3.2 (B)
- net VCC: now also AND-GATE-INT2.14 (VDD), AND-GATE-INT3.14 (VDD)
- net ~{INT_1``}: now also NOT-GATE-INT1.2 (~{1Y}); no longer NOT-GATE-INT1.4 (~{2Y})
- net ~{INT_3``_OR_INT_4``}: now also AND-GATE-INT1.8 (E), NOT-GATE-INT1.12 (~{6Y}), AND-GATE-INT3.5 (C); no longer NOT-GATE-INT1.2 (~{1Y})
- net INT_2``_AND_(~{INT_3``_OR_INT_4``}): now reaches AND-GATE-INT1.10 (L=E.F)
- net INT_2``_AND_(~{INT_3``_OR_INT_4``}): now also AND-GATE-INT2.8 (E)
- net INT_3``_AND_~{INT_4``}: now reaches AND-GATE-INT1.11 (M=G.H)
- net INT_3``_AND_~{INT_4``}: now also AND-GATE-INT2.6 (D)
- net ~{INT_4``}: now reaches AND-GATE-INT1.12 (G)
- net ~{INT_4``}: now also NOT-GATE-INT1.8 (~{4Y})
- net ~{INT_1``_OR_INT_2``}: now reaches NOT-GATE-INT1.10 (~{5Y})
- net ~{INT_1``_OR_INT_2``}: now also AND-GATE-INT3.6 (D)
- net RST_INT_ENABLE`: now reaches OR-GATE-RESETS1.10 (L=E+F)
- net RST_INT_ENABLE`: now also SR-LATCH-INTERRUPTS2.3 (R1)
- net INT_ADDRESS_OUT renamed ~{INT_ADDRESS_OUT}
- new net: AND-GATE-INT3.1 (A), AND-GATE-INT3.4 (K=C.D)
- new net: AND-GATE-INT3.11 (M=G.H), AND-GATE-INT3.9 (F)
- new net INT_1``_AND_~{INT_2``}_AND_(~{INT3``_OR_INT4``}): AND-GATE-INT2.13 (H), AND-GATE-INT3.10 (L=E.F)
- new net ~{INT3``_OR_INT4``}: AND-GATE-INT3.8 (E)
- new net ~{INT_2``}: AND-GATE-INT3.12 (G), NOT-GATE-INT1.4 (~{2Y})
- no-connect marks 131 -> 121
Other:
- moved on the sheet: AND-GATE-INT1, NOT-GATE-INT1, OR-GATE-INT1, TRNS-INT-ADDRESS1, TRNS-INT-ADDRESS2

Commit message: PCBs done
Parts:
- removed IDC-ADDRESS-BUS4, IDC-DATA-BUS4: DS1013-20SSIB1-B-0, Connector_PinSocket_2.54mm:PinSocket_2x10_P2.54mm_Vertical, symbol DS1013-20SSIB1-B-0:DS1013-20SSIB1-B-0
- added AND-GATE-SIGNALS1, AND-GATE-SIGNALS2, AND-GATE-SIGNALS3: CD4081BEE4, Package_DIP:DIP-14_W7.62mm, symbol CD4081BEE4:CD4081BEE4
- added BUTTON-OUT1: Conn-1x2, Connector_PinHeader_2.54mm:PinHeader_1x02_P2.54mm_Vertical, symbol Connector_Generic:Conn_01x02
- added BUTTON1, BUTTON1-TIMER2: SW_MEC_5E, Button_Switch_THT:SW_Push_2P1T_Toggle_CK_PVA1xxH1xxxxxxV2, symbol Switch:SW_MEC_5E
- added IDC-INT-DATA-BUS1, IDC-INT-DATA-BUS2: DS1013-20SSIB1-B-0, Connector_PinSocket_2.54mm:PinSocket_2x10_P2.54mm_Vertical, symbol DS1013-20SSIB1-B-0:DS1013-20SSIB1-B-0
- added LED_CLK1, LED_ID0, LED_ID1, LED_ID2, LED_ID3, LED_ID4, LED_ID5, LED_ID6, LED_ID7, LED_~{CLK}1: LED, LED_THT:LED_D5.0mm_FlatTop, symbol Device:LED
- added MODE-SELECTOR-2: SW_DPDT_x2, Button_Switch_THT:SW_Slide-03_Wuerth-WS-SLTV_10x2.5x6.4_P2.54mm, symbol Switch:SW_DPDT_x2
- added NOT-GATE-CLK1: CD74HC04E, Package_DIP:DIP-14_W7.62mm, symbol CD74HC04E:CD74HC04E
- added OR-GATE-INT-DATA1: CD4071BEE4, Package_DIP:DIP-14_W7.62mm, symbol CD4071BEE4:CD4071BEE4
- added REG-INT-DATA1: SN74HC574N, Package_DIP:DIP-20_W7.62mm, symbol SN74HC574N:SN74HC574N
- added R_CLK1, R_DOWN2, R_DOWN4, R_ID0, R_ID1, R_ID2, R_ID3, R_ID4, R_ID5, R_ID6, R_ID7, R_~{CLK}1, TIMER1-R1, TIMER1-R2, TIMER2-R1: R_US, Resistor_THT:R_Axial_DIN0204_L3.6mm_D1.6mm_P7.62mm_Horizontal, symbol Device:R_US
- added TIMER1, TIMER2: LMC555xN, Package_DIP:DIP-8_W7.62mm, symbol Timer:LMC555xN
- added TIMER1-C1, TIMER1-C2, TIMER2-C1, TIMER2-C2: C, Capacitor_THT:C_Disc_D3.0mm_W1.6mm_P2.50mm, symbol Device:C
- added TIMER1-C3, TIMER1-C4: C_Polarized_US, Capacitor_THT:CP_Radial_D5.0mm_P2.50mm, symbol Device:C_Polarized_US
- added TRNS-INT-DATA1: SN74AC245N, Package_DIP:DIP-20_W7.62mm, symbol SN74AC245N:SN74AC245N
Connections:
- net DATA0: now also TRNS-INT-DATA1.11 (B8)
- net DATA1: now also TRNS-INT-DATA1.12 (B7)
- net DATA2: now also TRNS-INT-DATA1.13 (B6)
- net DATA3: now also TRNS-INT-DATA1.14 (B5)
- net DATA4: now also TRNS-INT-DATA1.15 (B4)
- net DATA5: now also TRNS-INT-DATA1.16 (B3)
- net DATA6: now also TRNS-INT-DATA1.17 (B2)
- net DATA7: now also TRNS-INT-DATA1.18 (B1)
- net GND: now also AND-GATE-SIGNALS1.7 (VSS), AND-GATE-SIGNALS2.7 (VSS), AND-GATE-SIGNALS3.7 (VSS), LED_CLK1.1 (K), LED_ID0.1 (K), LED_ID1.1 (K), LED_ID2.1 (K), LED_ID3.1 (K), LED_ID4.1 (K), LED_ID5.1 (K), LED_ID6.1 (K), LED_ID7.1 (K), LED_~{CLK}1.1 (K), NOT-GATE-CLK1.7 (GND), OR-GATE-INT-DATA1.7 (VSS), REG-INT-DATA1.1 (~{OE}), REG-INT-DATA1.10 (GND), R_DOWN2.2, R_DOWN4.2, TIMER1-C1.2, TIMER1-C2.2, TIMER1-C3.2, TIMER1-C4.2, TIMER1.1 (GND), TIMER2-C1.2, TIMER2-C2.2, TIMER2.1 (GND), TRNS-INT-DATA1.10 (GND)
- net MCC_TICK: now also AND-GATE-SIGNALS3.10 (L=E.F); no longer BUFFER-F1.18 (2Q)
- net PC_TICK: now also AND-GATE-SIGNALS2.10 (L=E.F); no longer BUFFER-C1.13 (7Q)
- net REG_A_LOAD: now also AND-GATE-SIGNALS1.3 (J=A.B); no longer BUFFER-A1.19 (1Q)
- net REG_B_LOAD: now also AND-GATE-SIGNALS1.4 (K=C.D); no longer BUFFER-A1.18 (2Q)
- net REG_F_LOAD: now also AND-GATE-SIGNALS1.11 (M=G.H); no longer BUFFER-A1.12 (8Q)
- net REG_IR_LOAD: now also AND-GATE-SIGNALS3.11 (M=G.H); no longer BUFFER-F1.19 (1Q)
- net REG_MAR_LOAD: now also AND-GATE-SIGNALS3.3 (J=A.B); no longer BUFFER-D1.14 (6Q)
- net REG_MBR_LOAD: now also AND-GATE-SIGNALS3.4 (K=C.D); no longer BUFFER-D1.13 (7Q)
- net REG_TMPH_LOAD: now also AND-GATE-SIGNALS2.3 (J=A.B); no longer BUFFER-B1.17 (3Q)
- net REG_TMPL_LOAD: now also AND-GATE-SIGNALS2.4 (K=C.D); no longer BUFFER-B1.16 (4Q)
- net RST_INT_ENABLE: now also OR-GATE-RESETS1.10 (L=E+F), SR-LATCH-INTERRUPTS2.3 (R1); no longer BUFFER-G1.18 (2Q), OR-GATE-RESETS1.8 (E)
- net RST_INT_ENABLE`: now also BUFFER-G1.18 (2Q), OR-GATE-RESETS1.8 (E); no longer OR-GATE-RESETS1.10 (L=E+F), SR-LATCH-INTERRUPTS2.3 (R1)
- net STC_TICK: now also AND-GATE-SIGNALS2.11 (M=G.H); no longer BUFFER-D1.17 (3Q)
- net VCC: now also AND-GATE-SIGNALS1.14 (VDD), AND-GATE-SIGNALS2.14 (VDD), AND-GATE-SIGNALS3.14 (VDD), BUTTON1-TIMER2.2, BUTTON1.2, NOT-GATE-CLK1.14 (VCC), OR-GATE-INT-DATA1.14 (VDD), REG-INT-DATA1.20 (VCC), TIMER1-C1.1, TIMER1-R1.1, TIMER1.4 (R), TIMER1.8 (VCC), TIMER2-C1.1, TIMER2-R1.1, TIMER2.4 (R), TIMER2.8 (VCC), TRNS-INT-DATA1.1 (DIR), TRNS-INT-DATA1.20 (VCC)
- net ~{CLK}: now also AND-GATE-SIGNALS1.12 (G), AND-GATE-SIGNALS1.2 (B), AND-GATE-SIGNALS1.5 (C), AND-GATE-SIGNALS2.12 (G), AND-GATE-SIGNALS2.2 (B), AND-GATE-SIGNALS2.5 (C), AND-GATE-SIGNALS2.9 (F), AND-GATE-SIGNALS3.2 (B), AND-GATE-SIGNALS3.5 (C), NOT-GATE-CLK1.2 (~{1Y}), R_~{CLK}1.1
- net ~{INT_DATA_OUT}: now reaches BUFFER-G1.16 (4Q)
- net ~{INT_DATA_OUT}: now also TRNS-INT-DATA1.19 (~{OE})
- new net: TIMER1-R1.2, TIMER1-R2.1, TIMER1.7 (DIS)
- new net: TIMER1-C4.1, TIMER2-R1.2, TIMER2.6 (THR), TIMER2.7 (DIS)
- new net: LED_ID0.2 (A), R_ID0.2
- new net: LED_ID3.2 (A), R_ID3.2
- new net: LED_ID6.2 (A), R_ID6.2
- new net: TIMER1-C3.1, TIMER1-R2.2, TIMER1.2 (TR), TIMER1.6 (THR)
- new net: MODE-SELECTOR-2.1 (A), TIMER1.3 (Q)
- new net: TIMER1-C2.1, TIMER1.5 (CV)
- new net: LED_ID1.2 (A), R_ID1.2
- new net: BUTTON-OUT1.1 (Pin_1), BUTTON-OUT1.2 (Pin_2), BUTTON1.4 (A)
- new net: LED_ID5.2 (A), R_ID5.2
- new net: OR-GATE-INT-DATA1.10 (L=E+F), REG-INT-DATA1.11 (CLK)
- new net: LED_~{CLK}1.2 (A), R_~{CLK}1.2
- new net: BUTTON1-TIMER2.4 (A), TIMER2.2 (TR)
- new net: MODE-SELECTOR-2.3 (C), TIMER2.3 (Q)
- new net: TIMER2-C2.1, TIMER2.5 (CV)
- new net: BUTTON1-TIMER2.3 (K), R_DOWN4.1
- new net: LED_ID7.2 (A), R_ID7.2
- new net: BUTTON1.3 (K), R_DOWN2.1
- new net: LED_ID2.2 (A), R_ID2.2
- new net: LED_CLK1.2 (A), R_CLK1.2
- new net: LED_ID4.2 (A), R_ID4.2
- new net CLK: AND-GATE-SIGNALS3.12 (G), AND-GATE-SIGNALS3.9 (F), MODE-SELECTOR-2.2 (B), NOT-GATE-CLK1.1 (1A), R_CLK1.1
- new net INT_DATA0: REG-INT-DATA1.12 (8Q), R_ID0.1, TRNS-INT-DATA1.9 (A8)
- new net INT_DATA1: REG-INT-DATA1.13 (7Q), R_ID1.1, TRNS-INT-DATA1.8 (A7)
- new net INT_DATA2: REG-INT-DATA1.14 (6Q), R_ID2.1, TRNS-INT-DATA1.7 (A6)
- new net INT_DATA3: REG-INT-DATA1.15 (5Q), R_ID3.1, TRNS-INT-DATA1.6 (A5)
- new net INT_DATA4: REG-INT-DATA1.16 (4Q), R_ID4.1, TRNS-INT-DATA1.5 (A4)
- new net INT_DATA5: REG-INT-DATA1.17 (3Q), R_ID5.1, TRNS-INT-DATA1.4 (A3)
- new net INT_DATA6: REG-INT-DATA1.18 (2Q), R_ID6.1, TRNS-INT-DATA1.3 (A2)
- new net INT_DATA7: REG-INT-DATA1.19 (1Q), R_ID7.1, TRNS-INT-DATA1.2 (A1)
- new net INT_DATA_IN_0: IDC-INT-DATA-BUS1.19, IDC-INT-DATA-BUS1.20, IDC-INT-DATA-BUS2.19, IDC-INT-DATA-BUS2.20, REG-INT-DATA1.9 (8D)
- new net INT_DATA_IN_1: IDC-INT-DATA-BUS1.17, IDC-INT-DATA-BUS1.18, IDC-INT-DATA-BUS2.17, IDC-INT-DATA-BUS2.18, REG-INT-DATA1.8 (7D)
- new net INT_DATA_IN_2: IDC-INT-DATA-BUS1.15, IDC-INT-DATA-BUS1.16, IDC-INT-DATA-BUS2.15, IDC-INT-DATA-BUS2.16, REG-INT-DATA1.7 (6D)
- new net INT_DATA_IN_3: IDC-INT-DATA-BUS1.13, IDC-INT-DATA-BUS1.14, IDC-INT-DATA-BUS2.13, IDC-INT-DATA-BUS2.14, REG-INT-DATA1.6 (5D)
- new net INT_DATA_IN_4: IDC-INT-DATA-BUS1.11, IDC-INT-DATA-BUS1.12, IDC-INT-DATA-BUS2.11, IDC-INT-DATA-BUS2.12, REG-INT-DATA1.5 (4D)
- new net INT_DATA_IN_5: IDC-INT-DATA-BUS1.10, IDC-INT-DATA-BUS1.9, IDC-INT-DATA-BUS2.10, IDC-INT-DATA-BUS2.9, REG-INT-DATA1.4 (3D)
- new net INT_DATA_IN_6: IDC-INT-DATA-BUS1.7, IDC-INT-DATA-BUS1.8, IDC-INT-DATA-BUS2.7, IDC-INT-DATA-BUS2.8, REG-INT-DATA1.3 (2D)
- new net INT_DATA_IN_7: IDC-INT-DATA-BUS1.5, IDC-INT-DATA-BUS1.6, IDC-INT-DATA-BUS2.5, IDC-INT-DATA-BUS2.6, REG-INT-DATA1.2 (1D)
- new net MCC_TICK`: AND-GATE-SIGNALS3.8 (E), BUFFER-F1.18 (2Q)
- new net PC_TICK`: AND-GATE-SIGNALS2.8 (E), BUFFER-C1.13 (7Q)
- new net REG_A_LOAD`: AND-GATE-SIGNALS1.1 (A), BUFFER-A1.19 (1Q)
- new net REG_B_LOAD`: AND-GATE-SIGNALS1.6 (D), BUFFER-A1.18 (2Q)
- new net REG_F_LOAD`: AND-GATE-SIGNALS1.13 (H), BUFFER-A1.12 (8Q)
- new net REG_INT_DATA_LOAD1: IDC-INT-DATA-BUS1.3, IDC-INT-DATA-BUS1.4, OR-GATE-INT-DATA1.9 (F)
- new net REG_INT_DATA_LOAD2: IDC-INT-DATA-BUS2.3, IDC-INT-DATA-BUS2.4, OR-GATE-INT-DATA1.8 (E)
- new net REG_IR_LOAD`: AND-GATE-SIGNALS3.13 (H), BUFFER-F1.19 (1Q)
- new net REG_MAR_LOAD`: AND-GATE-SIGNALS3.1 (A), BUFFER-D1.14 (6Q)
- new net REG_MBR_LOAD`: AND-GATE-SIGNALS3.6 (D), BUFFER-D1.13 (7Q)
- new net REG_TMPH_LOAD`: AND-GATE-SIGNALS2.1 (A), BUFFER-B1.17 (3Q)
- new net REG_TMPL_LOAD`: AND-GATE-SIGNALS2.6 (D), BUFFER-B1.16 (4Q)
- new net STC_TICK`: AND-GATE-SIGNALS2.13 (H), BUFFER-D1.17 (3Q)
- no-connect marks 121 -> 140
Other:
- moved on the sheet: AND-GATE-INT1, AND-GATE-INT2, AND-GATE-INT3, AND-GATE-SELECTOR1, BOOT-MODE1, BUFFER-A1, BUFFER-B1, BUFFER-C1, BUFFER-D1, BUFFER-E1, BUFFER-F1, BUFFER-G1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
