File: schematics/final-alu/final-alu.kicad_pcb (KiCad board)
At the start: 2 copper layers, 200 x 300 mm, 112 parts

Commit message: PCBs done
Parts:
- added G***: LOGO, additional-libraries:bb-logo, F.Cu at (74.0, 82.0)
Routing:
- net FLAG7: track 115.7 -> 127.7 mm
- added copper zone on B.Cu, net GND
- added copper zone on F.Cu, net GND
Other:
- outline, holes or cut-outs redrawn
- board text added: "2024"

Commit message: Generated gerber files
Routing:
- net GND: vias 43 -> 107
